File: carte-io/hardware/carte-io/cpu.kicad_sch (KiCad schematic)
At the start: 21 parts, among them J3 FTSH-110-01-L-DV-007, U1 STM32U545VETx, X1 ASE-16.000MHZ-LC-T

Commit message: Carte IO routée version 1
Parts:
- added R72: 10K, Resistor_SMD:R_0805_2012Metric_Pad1.20x1.40mm_HandSolder, symbol Device:R
- added SW1, SW2: SW_Push, Button_Switch_THT:SW_TH_Tactile_Omron_B3F-10xx, symbol Switch:SW_Push
- J3: value FTSH-110-01-L-DV-007 -> FTSH-105-01-L-DV-007; footprint FTSH-105-X-X-DV-007-P-X:SAMTEC_FTSH-105-X-X-DV-007-P-X -> FTSH-105-01-L-DV-007-K:SAMTEC_FTSH-105-X-X-DV-007-P-X
- R2: value 100R -> 10K
- R28: value 100R -> 1K
Connections:
- net GND: now also SW1.1, SW2.1
- net NRST: now also R72.1
- net USER_BTN: now also SW1.2
- net JTDI: no longer names the net of U1.77 (PA15)
- net JTRST: no longer names the net of U1.90 (PB4)
- net SPI_CS1 renamed SPI_CS
- net SPI_CS2: no longer names the net of U1.98 (PE1)
- net SPI_CS3: no longer names the net of U1.1 (PE2)
- new net: R72.2, SW2.2
- no-connect marks 14 -> 18
Other:
- title: cpu (carte-io) -> CPU
