File: carte-io/hardware/carte-io/externals_i2c.kicad_sch (KiCad schematic)
At the start: 15 parts, among them J10 JST_PH_B4B, J11 JST_PH_B4B, J12 JST_PH_B4B, J13 JST_PH_B4B, J14 JST_PH_B4B, J15 JST_PH_B4B, J16 JST_PH_B4B, J17 JST_PH_B4B, J25 JST_PH_B4B, U15 PCA9544APW, U17 PCA9544APW, U33 MCP2542FDxMF

Commit message: Carte IO routée version 1
Parts:
- added C35, C36: 100nF, Capacitor_SMD:C_0805_2012Metric_Pad1.18x1.45mm_HandSolder, symbol Device:C
- added J23, J24: JST_PH_B4B, Connector_JST:JST_PH_B4B-PH-K_1x04_P2.00mm_Vertical, symbol Connector_Generic:Conn_01x04
- added R54, R55, R56, R57, R58, R59, R60, R61, R62, R63, R64, R65, R66, R67, R68, R69, R70, R71: 1K, Resistor_SMD:R_0805_2012Metric_Pad1.20x1.40mm_HandSolder, symbol Device:R
- added U35: TCA9802, Package_SO:VSSOP-8_3x3mm_P0.65mm, symbol Interface:TCA9802
Connections:
- net +3.3V: now also C35.1, C36.1, R54.1, R55.1, R56.1, R57.1, R58.1, R59.1, R60.1, R61.1, R62.2, R63.2, R64.1, R65.1, R66.1, R67.1, R68.1, R69.1, R70.2, R71.2, U35.1 (VCCA), U35.5 (EN), U35.8 (VCCB)
- net +3.3V_PWR: now also J23.1 (Pin_1), J24.1 (Pin_1)
- net GND: now also C35.2, C36.2, J23.3 (Pin_3), J24.3 (Pin_3), U35.4 (GND)
- net at J15.2 (Pin_2), U15.15 (SD3): now also R60.2
- net at J15.4 (Pin_4), U15.16 (SC3): now also R61.2
- net at J10.2 (Pin_2), U15.5 (SD0): now also R56.2
- net at J10.4 (Pin_4), U15.6 (SC0): now also R57.2
- net at J13.2 (Pin_2), U17.12 (SD2): now also R71.1
- net at J13.4 (Pin_4), U17.13 (SC2): now also R70.1
- net at J17.2 (Pin_2), U17.15 (SD3): now also R68.2
- net at J17.4 (Pin_4), U17.16 (SC3): now also R69.2
- net at J12.2 (Pin_2), U17.5 (SD0): now also R64.2
- net at J12.4 (Pin_4), U17.6 (SC0): now also R65.2
- net at J16.2 (Pin_2), U17.8 (SD1): now also R66.2
- net at J16.4 (Pin_4), U17.9 (SC1): now also R67.2
- net at J14.2 (Pin_2), U15.8 (SD1): now also R58.2
- net at J14.4 (Pin_4), U15.9 (SC1): now also R59.2
- net at J11.2 (Pin_2), U15.12 (SD2): now also R63.1
- net at J11.4 (Pin_4), U15.13 (SC2): now also R62.1
- new net: J23.2 (Pin_2), J24.2 (Pin_2), U35.6 (SDAB)
- new net: J23.4 (Pin_4), J24.4 (Pin_4), U35.7 (SCLB)
- new net I2C_SCL_ARBITRARY: R54.2, U35.2 (SCLA)
- new net I2C_SDA_ARBITRARY: R55.2, U35.3 (SDAA)
Other:
- company: (none) -> INSA - GEI
- title: (none) -> Externals I2C
- moved on the sheet: J10, J11, J12, J13, J14, J15, J16, J17, U17
