File: carte-io/hardware/carte-io/externals_i2c.kicad_sch (KiCad schematic)
At the start: 38 parts, among them J10 JST_PH_B4B, J11 JST_PH_B4B, J12 JST_PH_B4B, J13 JST_PH_B4B, J14 JST_PH_B4B, J15 JST_PH_B4B, J16 JST_PH_B4B, J17 JST_PH_B4B, J23 JST_PH_B4B, J24 JST_PH_B4B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

Commit message: Carte version 1.1 terminée
Parts:
- added R73, R74, R76, R77: 4.7K, Resistor_SMD:R_0805_2012Metric_Pad1.20x1.40mm_HandSolder, symbol Device:R
- J10, J11, J16, J17, J23, J24, J25: value JST_PH_B4B -> 114020164; footprint Connector_JST:JST_PH_B4B-PH-K_1x04_P2.00mm_Vertical -> SeeedStudio - Horizontal Header -114020164:SEEEDSTUDIO_114020164; symbol Connector_Generic:Conn_01x04 -> SeeedStudio - Horizontal header:SeeedStudio - 114020164 - R/A
- J12: renamed from J14; value JST_PH_B4B -> 114020164; footprint Connector_JST:JST_PH_B4B-PH-K_1x04_P2.00mm_Vertical -> SeeedStudio - Horizontal Header -114020164:SEEEDSTUDIO_114020164; symbol Connector_Generic:Conn_01x04 -> SeeedStudio - Horizontal header:SeeedStudio - 114020164 - R/A
- J13: renamed from J15; value JST_PH_B4B -> 114020164; footprint Connector_JST:JST_PH_B4B-PH-K_1x04_P2.00mm_Vertical -> SeeedStudio - Horizontal Header -114020164:SEEEDSTUDIO_114020164; symbol Connector_Generic:Conn_01x04 -> SeeedStudio - Horizontal header:SeeedStudio - 114020164 - R/A
- J14: renamed from J12; value JST_PH_B4B -> 114020164; footprint Connector_JST:JST_PH_B4B-PH-K_1x04_P2.00mm_Vertical -> SeeedStudio - Horizontal Header -114020164:SEEEDSTUDIO_114020164; symbol Connector_Generic:Conn_01x04 -> SeeedStudio - Horizontal header:SeeedStudio - 114020164 - R/A
- J15: renamed from J13; value JST_PH_B4B -> 114020164; footprint Connector_JST:JST_PH_B4B-PH-K_1x04_P2.00mm_Vertical -> SeeedStudio - Horizontal Header -114020164:SEEEDSTUDIO_114020164; symbol Connector_Generic:Conn_01x04 -> SeeedStudio - Horizontal header:SeeedStudio - 114020164 - R/A
- R54, R55, R56, R57, R58, R59, R60, R61, R62, R63, R64, R65, R66, R67, R68, R69, R70, R71: value 1K -> 4.7K
Connections:
- net +3.3V: now also R73.1, R74.1, R76.1, R77.1
- net +3.3V_PWR: now also J10.3 (Pin_3), J11.3 (Pin_3), J12.3 (Pin_3), J13.3 (Pin_3), J14.3 (Pin_3), J15.3 (Pin_3), J16.3 (Pin_3), J17.3 (Pin_3), J23.3 (Pin_3), J24.3 (Pin_3); no longer J10.1 (Pin_1), J11.1 (Pin_1), J12.1 (Pin_1), J13.1 (Pin_1), J14.1 (Pin_1), J15.1 (Pin_1), J16.1 (Pin_1), J17.1 (Pin_1), J23.1 (Pin_1), J24.1 (Pin_1)
- net +5V: now also J25.3 (Pin_3); no longer J25.1 (Pin_1)
- net GND: now also J10.4 (Pin_4), J11.4 (Pin_4), J12.4 (Pin_4), J13.4 (Pin_4), J14.4 (Pin_4), J15.4 (Pin_4), J16.4 (Pin_4), J17.4 (Pin_4), J23.4 (Pin_4), J24.4 (Pin_4), J25.4 (Pin_4); no longer J10.3 (Pin_3), J11.3 (Pin_3), J12.3 (Pin_3), J13.3 (Pin_3), J14.3 (Pin_3), J15.3 (Pin_3), J16.3 (Pin_3), J17.3 (Pin_3), J23.3 (Pin_3), J24.3 (Pin_3), J25.3 (Pin_3)
- net SENSORS_I2C_SCL: now also R76.2
- net SENSORS_I2C_SDA: now also R77.2
- net at R67.2, U17.9 (SC1): now also J16.1 (Pin_1); no longer J16.4 (Pin_4)
- net at J23.2 (Pin_2), J24.2 (Pin_2), U35.6 (SDAB): now also R74.2
- net at R61.2, U15.16 (SC3): now also J13.1 (Pin_1); no longer J13.4 (Pin_4)
- net at R57.2, U15.6 (SC0): now also J10.1 (Pin_1); no longer J10.4 (Pin_4)
- net at R69.2, U17.16 (SC3): now also J17.1 (Pin_1); no longer J17.4 (Pin_4)
- net at R70.1, U17.13 (SC2): now also J15.1 (Pin_1); no longer J15.4 (Pin_4)
- net at R65.2, U17.6 (SC0): now also J14.1 (Pin_1); no longer J14.4 (Pin_4)
- net at R35.2, U33.6 (CANL): now also J25.1 (Pin_1); no longer J25.4 (Pin_4)
- net at R59.2, U15.9 (SC1): now also J12.1 (Pin_1); no longer J12.4 (Pin_4)
- net at R62.1, U15.13 (SC2): now also J11.1 (Pin_1); no longer J11.4 (Pin_4)
- new net: J23.1 (Pin_1), J24.1 (Pin_1), R73.2, U35.7 (SCLB)
Other:
- moved on the sheet: J23, J24, R35, R66, R67, R68, R69
