File: carte-io/hardware/carte-io/int_sensors.kicad_sch (KiCad schematic)
At the start: 22 parts, among them U12 LSM6DS3, U13 LIS2MDL, U14 LPS22DF, U18 APDS-9251-001, U19 SHT4x

Commit message: Carte IO routée version 1
Parts:
- removed C22, C23, C24, C25, C26, C27, C28, C29, C35, C36: 100nF, Capacitor_SMD:C_0805_2012Metric_Pad1.18x1.45mm_HandSolder, symbol Device:C
- R29, R30: value 10K -> 1K
Other:
- company: (none) -> INSA GEI
- title: (none) -> Internals sensors
