File: carte-io/hardware/carte-io/int_sensors.kicad_sch (KiCad schematic)
At the start: 12 parts, among them U12 LSM6DS3, U13 LIS2MDL, U14 LPS22DF, U18 APDS-9251-001, U19 SHT4x

Commit message: Carte version 1.1 terminée
Parts:
- R29, R30: value 1K -> 4.7K
Changed lines of the file:
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@@
 	(title_block
 		(title "Internals sensors")
-		(date "2024-11-05")
-		(rev "1.0")
+		(date "2025-02-25")
+		(rev "1.1")
 		(company "INSA GEI")
 	)
@@
 			)
 		)
-		(property "Value" "1K"
+		(property "Value" "4.7K"
 			(at 60.96 34.2899 0)
 			(effects
@@
 			)
 		)
-		(property "Value" "1K"
+		(property "Value" "4.7K"
 			(at 50.8 34.2899 0)
 			(effects
