File: carte-io/hardware/carte-io/motors.kicad_sch (KiCad schematic)
At the start: 30 parts, among them J4 JST_PH_B4B, J5 JST_PH_B4B, J6 JST_PH_B4B, J7 JST_PH_B4B, J8 TSW-104-07-G-T, J9 TSW-104-07-G-T, U10 CM1293A-04SO, U11 74LVC125APW, U4 CM1293A-04SO, U5 TXU0104PWR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

Commit message: Carte IO routée version 1
Connections:
- no-connect marks 0 -> 2
Other:
- company: (none) -> INSA - GEI
- title: (none) -> Motors & Servo
Changed lines of the file:
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@@
 	(generator_version "8.0")
 	(paper "A4")
+	(title_block
+		(title "Motors & Servo")
+		(date "2024-11-05")
+		(rev "1.0")
+		(company "INSA - GEI")
+	)
 	(junction
 		(at 236.22 58.42)
@@
 		(color 0 0 0 0)
 	)
+	(no_connect
+		(at 207.01 66.04)
+	)
+	(no_connect
+		(at 77.47 62.23)
+	)
 	(wire
 		(pts
@@
 	)
 	(hierarchical_label "ENCODER_4_PHB"
-		(shape input)
+		(shape output)
 		(at 246.38 132.08 0)
 		(fields_autoplaced yes)
@@
 	)
 	(hierarchical_label "ENCODER_3_PHB"
-		(shape input)
+		(shape output)
 		(at 246.38 127 0)
 		(fields_autoplaced yes)
@@
 	)
 	(hierarchical_label "ENCODER_3_PHA"
-		(shape input)
+		(shape output)
 		(at 246.38 124.46 0)
 		(fields_autoplaced yes)
@@
 	)
 	(hierarchical_label "ENCODER_1_PHB"
-		(shape input)
+		(shape output)
 		(at 111.76 125.73 0)
 		(fields_autoplaced yes)
@@
 	)
 	(hierarchical_label "ENCODER_1_PHA"
-		(shape input)
+		(shape output)
 		(at 111.76 123.19 0)
 		(fields_autoplaced yes)
@@
 	)
 	(hierarchical_label "ENCODER_2_PHA"
-		(shape input)
+		(shape output)
 		(at 111.76 128.27 0)
 		(fields_autoplaced yes)
@@
 	)
 	(hierarchical_label "ENCODER_2_PHB"
-		(shape input)
+		(shape output)
 		(at 111.76 130.81 0)
 		(fields_autoplaced yes)
@@
 	)
 	(hierarchical_label "ENCODER_4_PHA"
-		(shape input)
+		(shape output)
 		(at 246.38 129.54 0)
 		(fields_autoplaced yes)
@@
 		(dnp no)
 		(property "Reference" "R16"
-			(at 106.6799 49.53 0)
+			(at 104.902 51.816 90)
 			(effects
 				(font
@@
 		)
 		(property "Value" "100R"
-			(at 109.2199 49.53 0)
+			(at 117.094 52.07 90)
 			(effects
 				(font
@@
 		(dnp no)
 		(property "Reference" "R12"
-			(at 40.6399 123.19 0)
+			(at 42.926 128.27 90)
 			(effects
 				(font
@@
 		)
 		(property "Value" "100R"
-			(at 43.1799 123.19 0)
+			(at 44.196 130.302 90)
 			(effects
 				(font
@@
 		(dnp no)
 		(property "Reference" "R23"
-			(at 214.6299 50.8 0)
+			(at 216.916 49.022 90)
 			(effects
 				(font
@@
 		)
 		(property "Value" "100R"
-			(at 217.1699 50.8 0)
+			(at 218.186 50.8 90)
 			(effects
 				(font
@@
 		(dnp no)
 		(property "Reference" "R13"
-			(at 40.6399 147.32 0)
+			(at 42.926 145.288 90)
 			(effects
 				(font
@@
 		)
 		(property "Value" "100R"
-			(at 43.1799 147.32 0)
+			(at 44.196 147.066 90)
 			(effects
 				(font
@@
 		(dnp no)
 		(property "Reference" "R25"
-			(at 214.6299 55.88 0)
+			(at 211.836 58.42 90)
 			(effects
 				(font
@@
 		)
 		(property "Value" "100R"
-			(at 217.1699 55.88 0)
+			(at 225.298 58.42 90)
 			(effects
 				(font
@@
 		(dnp no)
 		(property "Reference" "R14"
-			(at 40.6399 152.4 0)
+			(at 42.926 157.734 90)
 			(effects
 				(font
@@
 		)
 		(property "Value" "100R"
-			(at 43.1799 152.4 0)
+			(at 44.196 159.766 90)
 			(effects
 				(font
@@
 		(dnp no)
 		(property "Reference" "R24"
-			(at 214.6299 53.34 0)
+			(at 211.836 55.88 90)
 			(effects
 				(font
@@
 		)
 		(property "Value" "100R"
-			(at 217.1699 53.34 0)
+			(at 225.044 55.88 90)
 			(effects
 				(font
@@
 		(dnp no)
 		(property "Reference" "R22"
-			(at 177.7999 153.67 0)
+			(at 180.086 158.496 90)
 			(effects
 				(font
@@
 		)
 		(property "Value" "100R"
-			(at 180.3399 153.67 0)
+			(at 181.356 160.528 90)
 			(effects
 				(font
@@
 		(dnp no)
 		(property "Reference" "R18"
-			(at 106.6799 54.61 0)
+			(at 108.966 59.69 90)
 			(effects
 				(font
@@
 		)
 		(property "Value" "100R"
-			(at 109.2199 54.61 0)
+			(at 110.236 61.468 90)
 			(effects
 				(font
@@
 		(dnp no)
 		(property "Reference" "R17"
-			(at 106.6799 52.07 0)
+			(at 104.902 54.61 90)
 			(effects
 				(font
@@
 		)
 		(property "Value" "100R"
-			(at 109.2199 52.07 0)
+			(at 117.094 54.61 90)
 			(effects
 				(font
@@
 		(dnp no)
 		(property "Reference" "R15"
-			(at 106.6799 46.99 0)
+			(at 108.712 44.45 90)
 			(effects
 				(font
@@
 		)
 		(property "Value" "100R"
-			(at 109.2199 46.99 0)
+			(at 109.982 47.244 90)
 			(effects
 				(font
@@
 		(dnp no)
 		(property "Reference" "R26"
-			(at 214.6299 58.42 0)
+			(at 217.17 63.754 90)
 			(effects
 				(font
@@
 		)
 		(property "Value" "100R"
-			(at 217.1699 58.42 0)
+			(at 218.44 65.786 90)
 			(effects
 				(font
@@
 		(dnp no)
 		(property "Reference" "R21"
-			(at 177.7999 148.59 0)
+			(at 180.086 146.304 90)
 			(effects
 				(font
@@
 		)
 		(property "Value" "100R"
-			(at 180.3399 148.59 0)
+			(at 181.356 148.59 90)
 			(effects
 				(font
@@
 		(dnp no)
 		(property "Reference" "R11"
-			(at 40.6399 118.11 0)
+			(at 42.926 115.57 90)
 			(effects
 				(font
@@
 		)
 		(property "Value" "100R"
-			(at 43.1799 118.11 0)
+			(at 44.196 118.11 90)
 			(effects
 				(font
@@
 		(dnp no)
 		(property "Reference" "R20"
-			(at 177.7999 124.46 0)
+			(at 180.34 129.54 90)
 			(effects
 				(font
@@
 		)
 		(property "Value" "100R"
-			(at 180.3399 124.46 0)
+			(at 181.61 131.572 90)
 			(effects
 				(font
@@
 		(dnp no)
 		(property "Reference" "R19"
-			(at 177.7999 119.38 0)
+			(at 180.086 117.348 90)
 			(effects
 				(font
@@
 		)
 		(property "Value" "100R"
-			(at 180.3399 119.38 0)
+			(at 181.356 119.38 90)
 			(effects
 				(font
