File: carte-io/hardware/carte-io/power_analog.kicad_sch (KiCad schematic)
At the start: 31 parts, among them J1 USB_C_Receptacle_USB2.0_14P, J2 JST-XH_S2B-XH-A, U16 LT1963AxST-3.3, U2 FT231XQ, U3 LT1963AxST-3.3

Commit message: Carte IO routée version 1
Parts:
- removed D3: D, Diode_SMD:D_2010_5025Metric, symbol Device:D
- removed F1: Polyfuse, Fuse:Fuse_Bourns_MF-RG300, symbol Device:Polyfuse
- added C22: 100nF, Capacitor_SMD:C_0805_2012Metric_Pad1.18x1.45mm_HandSolder, symbol Device:C
- added D9: BAT54SFILMY, Package_TO_SOT_SMD:SOT-23, symbol Diode:BAT54S
- added H1, H2, H3, H4: MountingHole, MountingHole:MountingHole_3.2mm_M3, symbol Mechanical:MountingHole
- added J26: JST-PH-B2B, Connector_JST:JST_PH_B2B-PH-K_1x02_P2.00mm_Vertical, symbol Connector_Generic:Conn_01x02
- added R52, R53: 100R, Resistor_SMD:R_0805_2012Metric_Pad1.20x1.40mm_HandSolder, symbol Device:R
- added R73, R74, R75: 5.1K, Resistor_SMD:R_0805_2012Metric_Pad1.20x1.40mm_HandSolder, symbol Device:R
- added U36: TPS259250DRCT, Package_SON:VSON-10-1EP_3x3mm_P0.5mm_EP1.65x2.4mm_ThermalVias, symbol Power_Management:TPS2592xx
- C17, C19, C21: value 100nF -> 10µF
- R7, R8: value 100R -> 1K
Connections:
- net +3.3V: now also D9.2 (K)
- net +5V: now also U36.6 (OUT), U36.7 (OUT), U36.8 (OUT)
- net GND: now also C22.2, D9.1 (A), J26.1 (Pin_1), R53.2, R74.2, R75.2, U36.11 (GND)
- net USB-DN: now reaches C15.1, J1.A6 (D+), J1.A7 (D-), R5.1
- net USB-DP: now reaches C14.1, J1.B6 (D+), J1.B7 (D-), R6.2
- net USB2-DN: now reaches R5.2, U2.12 (USBDM)
- net VIN: now reaches J2.2 (Pin_2)
- net VIN: now also R73.1, U36.3 (VIN), U36.4 (VIN), U36.5 (VIN)
- net USB2-DP: now reaches R6.1, U2.11 (USBDP)
- net FT231_VCC: now reaches FB1.2, U2.15 (VCC)
- new net: R75.1, U36.10 (ILIM)
- new net: J26.2 (Pin_2), R52.1
- new net: C22.1, U36.1 (dV/dT)
- new net: R73.2, R74.1, U36.2 (EN/UVLO)
- new net ADC_VBAT: D9.3 (COM), R52.2, R53.1
Other:
- note added: "5V => Puissance pour servomoteur 3.3V_PWR => 3.3v de puissance pour capteurs externes 3.3V => alimentation issue de l'USB pour alimentation du CPU et des capteurs internes VUSB => 5V issue de l'USB, transistoire vers 3.3V"
- title: Puissance (carte-io) -> Puissance
- moved on the sheet: C17, C18, C19, J2
