File: carte-io/hardware/carte-io/power_analog.kicad_sch (KiCad schematic)
At the start: 42 parts, among them J1 USB_C_Receptacle_USB2.0_14P, J2 JST-XH_S2B-XH-A, J26 JST-PH-B2B, U16 LT1963AxST-3.3, U2 FT231XQ, U3 LT1963AxST-3.3, U36 TPS259250DRCT

Commit message: Carte version 1.1 terminée
Parts:
- removed C17: 10µF, Capacitor_SMD:C_0805_2012Metric_Pad1.18x1.45mm_HandSolder, symbol Device:C
- removed C22: 100nF, Capacitor_SMD:C_0805_2012Metric_Pad1.18x1.45mm_HandSolder, symbol Device:C
- removed R73, R74, R75: 5.1K, Resistor_SMD:R_0805_2012Metric_Pad1.20x1.40mm_HandSolder, symbol Device:R
- removed U36: TPS259250DRCT, Package_SON:VSON-10-1EP_3x3mm_P0.5mm_EP1.65x2.4mm_ThermalVias, symbol Power_Management:TPS2592xx
- added JP3: Jumper_2_Bridged, Connector_PinHeader_2.54mm:PinHeader_1x02_P2.54mm_Horizontal, symbol Jumper:Jumper_2_Bridged
- added Q1: IRF9388TRPBF, Package_SO:SOIC-8_3.9x4.9mm_P1.27mm, symbol Transistor_FET:IRF7404
- J2: value JST-XH_S2B-XH-A -> 114020164; footprint Connector_JST:JST_XH_S2B-XH-A_1x02_P2.50mm_Horizontal -> SeeedStudio - Horizontal Header -114020164:SEEEDSTUDIO_114020164; symbol Connector_Generic:Conn_01x02 -> SeeedStudio - Horizontal header:SeeedStudio - 114020164 - R/A
- J26: value JST-PH-B2B -> 114020164; footprint Connector_JST:JST_PH_B2B-PH-K_1x02_P2.00mm_Vertical -> SeeedStudio - Horizontal Header -114020164:SEEEDSTUDIO_114020164; symbol Connector_Generic:Conn_01x02 -> SeeedStudio - Horizontal header:SeeedStudio - 114020164 - R/A
- R10, R27: value 100R -> 150R
- R7, R8: value 1K -> 150R
- R9: value 100R -> 330R
Connections:
- net +5V: now also JP3.2 (B)
- net GND: now also J2.4 (Pin_4), J26.4 (Pin_4), Q1.4 (G); no longer J26.1 (Pin_1)
- net USB-DN: now also J1.B7 (D-); no longer J1.A6 (D+)
- net USB-DP: now also J1.A6 (D+); no longer J1.B7 (D-)
- net VIN: now also J2.3 (Pin_3), Q1.5 (D), Q1.6 (D), Q1.7 (D), Q1.8 (D)
- net at R52.1: now also J26.3 (Pin_3); no longer J26.2 (Pin_2)
- new net: JP3.1 (A), Q1.1 (S), Q1.2 (S), Q1.3 (S)
- new net PWR_CSLEEP: J26.2 (Pin_2)
- new net ~{POWEROFF}: J26.1 (Pin_1)
Other:
- note added: "De base, le jumper JP3 est fermé, le 5V est fourni par le connecteur J2. Si le jumper est ouvert, le 5V est fourni par les controlleurs des moteurs."
- moved on the sheet: H2, H3, H4, R6
