File: carte-io/hardware/carte-io/uarts.kicad_sch (KiCad schematic)
At the start: 17 parts, among them J18 JST_PH_B4B, J19 JST_PH_B4B, J21 JST_PH_B4B, U20 74LVC2G125DP,125, U21 CM1293A-04SO, U26 74LVC2G125DP,125, U27 CM1293A-04SO, U28 74LVC2G125DP,125, U29 CM1293A-04SO

Commit message: Carte IO routée version 1
Parts:
- removed C0: 100nF, Capacitor_SMD:C_0805_2012Metric_Pad1.18x1.45mm_HandSolder, symbol Device:C
- removed R0: 100R, Resistor_SMD:R_0805_2012Metric_Pad1.20x1.40mm_HandSolder, symbol Device:R
Other:
- title: UARTS (carte-uarts) -> UARTS 
Changed lines of the file:
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@@
 	(paper "A4")
 	(title_block
-		(title "UARTS (carte-uarts)")
+		(title "UARTS ")
 		(date "2024-10-09")
 		(rev "1.0")
@@
 	)
 	(hierarchical_label "EXT_UART2_RX"
-		(shape input)
+		(shape output)
 		(at 171.45 71.12 180)
 		(fields_autoplaced yes)
@@
 	)
 	(hierarchical_label "EXT_UART1_RX"
-		(shape input)
+		(shape output)
 		(at 35.56 71.12 180)
 		(fields_autoplaced yes)
@@
 	)
 	(hierarchical_label "EXT_UART3_RX"
-		(shape input)
+		(shape output)
 		(at 179.07 142.24 180)
 		(fields_autoplaced yes)
@@
 		(dnp no)
 		(property "Reference" "R33"
-			(at 245.1099 50.8 0)
+			(at 247.396 48.514 90)
 			(effects
 				(font
@@
 		)
 		(property "Value" "100R"
-			(at 247.6499 50.8 0)
+			(at 248.666 50.8 90)
 			(effects
 				(font
@@
 		(dnp no)
 		(property "Reference" "R45"
-			(at 252.7299 121.92 0)
+			(at 255.27 119.38 90)
 			(effects
 				(font
@@
 		)
 		(property "Value" "100R"
-			(at 255.2699 121.92 0)
+			(at 256.286 121.92 90)
 			(effects
 				(font
@@
 	)
 	(symbol
-		(lib_id "Device:C")
-		(at -3.81 201.93 0)
-		(unit 1)
-		(exclude_from_sim no)
-		(in_bom yes)
-		(on_board yes)
-		(dnp no)
-		(fields_autoplaced yes)
-		(property "Reference" "C0"
-			(at 0 200.6599 0)
-			(effects
-				(font
-					(size 1.27 1.27)
-				)
-				(justify left)
-			)
-		)
-		(property "Value" "100nF"
-			(at 0 203.1999 0)
-			(effects
-				(font
-					(size 1.27 1.27)
-				)
-				(justify left)
-			)
-		)
-		(property "Footprint" "Capacitor_SMD:C_0805_2012Metric_Pad1.18x1.45mm_HandSolder"
-			(at -2.8448 205.74 0)
-			(effects
-				(font
-					(size 1.27 1.27)
-				)
-				(hide yes)
-			)
-		)
-		(property "Datasheet" "~"
-			(at -3.81 201.93 0)
-			(effects
-				(font
-					(size 1.27 1.27)
-				)
-				(hide yes)
-			)
-		)
-		(property "Description" "Unpolarized capacitor"
-			(at -3.81 201.93 0)
-			(effects
-				(font
-					(size 1.27 1.27)
-				)
-				(hide yes)
-			)
-		)
-		(pin "2"
-		)
-		(pin "1"
-		)
-		(instances
-			(project "carte-io"
-				(path "/acbeee85-bee7-482c-b859-0ad6bf15d6be/e0769f15-5851-4dbe-85c4-fc3863520381"
-					(reference "C0")
-					(unit 1)
-				)
-			)
-		)
-	)
-	(symbol
 		(lib_id "Connector_Generic:Conn_01x04")
 		(at 130.81 53.34 0)
@@
 		(dnp no)
 		(property "Reference" "R34"
-			(at 251.4599 55.88 0)
+			(at 253.746 61.468 90)
 			(effects
 				(font
@@
 		)
 		(property "Value" "100R"
-			(at 253.9999 55.88 0)
+			(at 255.016 63.754 90)
 			(effects
 				(font
@@
 		(dnp no)
 		(property "Reference" "R31"
-			(at 107.9499 50.8 0)
+			(at 110.49 48.768 90)
 			(effects
 				(font
@@
 		)
 		(property "Value" "100R"
-			(at 110.4899 50.8 0)
+			(at 110.4899 50.8 90)
 			(effects
 				(font
@@
 		(dnp no)
 		(property "Reference" "R46"
-			(at 259.0799 127 0)
+			(at 261.62 132.588 90)
 			(effects
 				(font
@@
 		)
 		(property "Value" "100R"
-			(at 261.6199 127 0)
+			(at 262.89 134.874 90)
 			(effects
 				(font
@@
 		(dnp no)
 		(property "Reference" "R32"
-			(at 114.2999 55.88 0)
+			(at 116.586 61.468 90)
 			(effects
 				(font
@@
 		)
 		(property "Value" "100R"
-			(at 116.8399 55.88 0)
+			(at 117.602 64.008 90)
 			(effects
 				(font
@@
 					(unit 1)
 				)
-			)
-		)
-	)
-	(symbol
-		(lib_id "Device:R")
-		(at 41.91 213.36 90)
-		(unit 1)
-		(exclude_from_sim no)
-		(in_bom yes)
-		(on_board yes)
-		(dnp no)
-		(property "Reference" "R0"
-			(at 40.6399 210.82 0)
-			(effects
-				(font
-					(size 1.27 1.27)
-				)
-				(justify left)
-			)
-		)
-		(property "Value" "100R"
-			(at 43.1799 210.82 0)
-			(effects
-				(font
-					(size 1.27 1.27)
-				)
-				(justify left)
-			)
-		)
-		(property "Footprint" "Resistor_SMD:R_0805_2012Metric_Pad1.20x1.40mm_HandSolder"
-			(at 41.91 215.138 90)
-			(effects
-				(font
-					(size 1.27 1.27)
-				)
-				(hide yes)
-			)
-		)
-		(property "Datasheet" "~"
-			(at 41.91 213.36 0)
-			(effects
-				(font
-					(size 1.27 1.27)
-				)
-				(hide yes)
-			)
-		)
-		(property "Description" "Resistor"
-			(at 41.91 213.36 0)
-			(effects
-				(font
-					(size 1.27 1.27)
-				)
-				(hide yes)
-			)
-		)
-		(pin "1"
-		)
-		(pin "2"
-		)
-		(instances
-			(project "carte-io"
-				(path "/acbeee85-bee7-482c-b859-0ad6bf15d6be/e0769f15-5851-4dbe-85c4-fc3863520381"
-					(reference "R0")
-					(unit 1)
-				)

Commit message: Correction du 5V sur les UART (Lidar et GPS + Changement de conencteur J27 (GPS) pour rajouter le 5V et le 3V pour les IO
Parts:
- removed J21: JST_PH_B4B, Connector_JST:JST_PH_B4B-PH-K_1x04_P2.00mm_Vertical, symbol Connector_Generic:Conn_01x04
- added J27: JST_PH_B5B, Connector_JST:JST_PH_B5B-PH-K_1x05_P2.00mm_Vertical, symbol Connector_Generic:Conn_01x05
Connections:
- net +3.3V: now also J27.2 (Pin_2); no longer U21.5 (VP), U27.5 (VP), U29.5 (VP)
- net GND: now also J27.4 (Pin_4)
- net at R45.2: now also J27.3 (Pin_3)
- net at R46.2: now also J27.5 (Pin_5)
- net +3.3V_PWR renamed +5V
- net +5V: now also U21.5 (VP), U27.5 (VP), U29.5 (VP), J27.1 (Pin_1)
Other:
- note added: "3V3 only for IO"
- note added: "5V for power supply"
- note added: "GPS Connector"
