File: carte-io/hardware/carte-io/uarts.kicad_sch (KiCad schematic)
At the start: 15 parts, among them J18 JST_PH_B4B, J19 JST_PH_B4B, J27 JST_PH_B5B, U20 74LVC2G125DP,125, U21 CM1293A-04SO, U26 74LVC2G125DP,125, U27 CM1293A-04SO, U28 74LVC2G125DP,125, U29 CM1293A-04SO

Commit message: Carte version 1.1 terminée
Parts:
- J18, J19: value JST_PH_B4B -> 114020164; footprint Connector_JST:JST_PH_B4B-PH-K_1x04_P2.00mm_Vertical -> SeeedStudio - Horizontal Header -114020164:SEEEDSTUDIO_114020164; symbol Connector_Generic:Conn_01x04 -> SeeedStudio - Horizontal header:SeeedStudio - 114020164 - R/A
- J27: value JST_PH_B5B -> 114020164; footprint Connector_JST:JST_PH_B5B-PH-K_1x05_P2.00mm_Vertical -> SeeedStudio - Horizontal Header -114020164:SEEEDSTUDIO_114020164; symbol Connector_Generic:Conn_01x05 -> SeeedStudio - Horizontal header:SeeedStudio - 114020164 - R/A
- U20, U26, U28: footprint Package_SO:VSSOP-8_2.3x2mm_P0.5mm -> Package_SO:TSSOP-8_3x3mm_P0.65mm
Connections:
- net +3.3V: now also U21.5 (VP), U27.5 (VP), U29.5 (VP); no longer J27.2 (Pin_2)
- net +5V: now also J18.3 (Pin_3), J19.3 (Pin_3), J27.3 (Pin_3); no longer J18.1 (Pin_1), J19.1 (Pin_1), J27.1 (Pin_1), U21.5 (VP), U27.5 (VP), U29.5 (VP)
- net GND: now also J18.4 (Pin_4), J19.4 (Pin_4); no longer J18.3 (Pin_3), J19.3 (Pin_3)
- net at R34.2: now also J19.1 (Pin_1); no longer J19.4 (Pin_4)
- net at R45.2: now also J27.2 (Pin_2); no longer J27.3 (Pin_3)
- net at R32.2: now also J18.1 (Pin_1); no longer J18.4 (Pin_4)
- net at R46.2: now also J27.1 (Pin_1); no longer J27.5 (Pin_5)
Other:
- note added: "UARTS Connectors"
- note removed: "GPS Connector"
- moved on the sheet: R31, R32, R33, R34, R45, R46, U20A, U26A, U28A
