File: carte-io/hardware/carte-io/gpio_spi.kicad_sch (KiCad schematic)
At the start: 32 parts, among them J20 Conn_02x08_Odd_Even, J22 JST_PH_B6B, U22 CM1293A-04SO, U23 74LVC125APW, U24 CM1293A-04SO, U25 74LVC125APW, U30 74LVC125APW,118, U31 CM1293A-04SO, U32 74LVC2G125DP,125, U34 CM1293A-04SO

Commit message: Carte version 1.1 terminée
Parts:
- removed C39, C40, C41, C46: 100nF, Capacitor_SMD:C_0805_2012Metric_Pad1.18x1.45mm_HandSolder, symbol Device:C
- removed J20: Conn_02x08_Odd_Even, Connector_PinHeader_2.54mm:PinHeader_2x07_P2.54mm_Vertical, symbol Connector_Generic:Conn_02x07_Odd_Even
- removed J22: JST_PH_B6B, Connector_JST:JST_PH_B6B-PH-K_1x06_P2.00mm_Vertical, symbol Connector_Generic:Conn_01x06
- removed R38, R39, R44, R47, R48, R49, R50, R51: 100R, Resistor_SMD:R_0805_2012Metric_Pad1.20x1.40mm_HandSolder, symbol Device:R
- removed U22, U31, U34: CM1293A-04SO, CM1293A-04SO:SOT95P285X140-6N, symbol CM1293A-04SO:CM1293A-04SO
- removed U23, U25: 74LVC125APW, 74LVC125APW:IC_74LVC125APW, symbol 74LVC125APW:74LVC125APW
- removed U30: 74LVC125APW,118, Package_SO:TSSOP-14_4.4x5mm_P0.65mm, symbol 74xx:74LVC125
- removed U32: 74LVC2G125DP,125, Package_SO:VSSOP-8_2.3x2mm_P0.5mm, symbol 74xGxx:74LVC2G125
- added D3, D8: BAT54SFILMY, Package_TO_SOT_SMD:SOT-23, symbol Diode:BAT54S
- added J20, J21, J22, J28, J29, J30: 114020164, SeeedStudio - Horizontal Header -114020164:SEEEDSTUDIO_114020164, symbol SeeedStudio - Horizontal header:SeeedStudio - 114020164 - R/A
Connections:
- net +3.3V: now also D3.2 (K), D8.2 (K), J20.3 (Pin_3), J21.3 (Pin_3), J22.3 (Pin_3), J28.3 (Pin_3), J29.3 (Pin_3), J30.3 (Pin_3)
- net GND: now also D3.1 (A), D8.1 (A), J20.4 (Pin_4), J21.4 (Pin_4), J22.4 (Pin_4), J28.4 (Pin_4), J29.4 (Pin_4), J30.4 (Pin_4)
- net IN_OUT4: now reaches R43.1, U24.6 (CH4)
- net IN_OUT3: now reaches R42.1, U24.4 (CH3)
- net IN_OUT1: now reaches R40.1, U24.1 (CH1)
- net IN_OUT2: now reaches R41.1, U24.3 (CH2)
- net ADC_AN1: now reaches R36.2
- net ADC_AN1: now also D3.3 (COM)
- net ADC_AN2: now reaches R37.2
- net ADC_AN2: now also D8.3 (COM)
- net IN1 renamed AN1
- net AN1: now also J29.1 (Pin_1)
- net IN2: no longer names the net of R37.1
- net IN2: now also J30.1 (Pin_1)
- net OUT1 renamed IO1
- net IO1: now also J20.1 (Pin_1)
- net OUT2 renamed IO2
- net IO2: now also J28.1 (Pin_1)
- net OUT3 renamed IO3
- net IO3: now also J21.1 (Pin_1)
- net OUT4 renamed IO4
- net IO4: now also J22.1 (Pin_1)
- no-connect marks 2 -> 6
Other:
- moved on the sheet: C42, R40, R41, R42, R43, U24
