Commit message: fix: rotate lidar link, change launch file to launch new RPLidar node

File: raspberryPI3/ros2_ws/src/geicar_description/src/description/geicar_description.urdf (robot description, URDF)
Before this commit: robot geicar, 18 links, 17 joints
Joints:
- joint rplidar_joint: origin xyz=${rplidar_xoff} ${rplidar_yoff} ${rplidar_zoff} rpy=0 0 ${pi/2} -> xyz=${rplidar_xoff} ${rplidar_yoff} ${rplidar_zoff} rpy=${pi} 0 ${-pi/2}

Commit message: fix: rotate lidar link, change launch file to launch new RPLidar node

File: raspberryPI3/ros2_ws/src/geicar_description/src/description/geicar_description.urdf (robot description, URDF)
Before this commit: robot geicar, 18 links, 17 joints
Joints:
- joint rplidar_joint: origin xyz=${rplidar_xoff} ${rplidar_yoff} ${rplidar_zoff} rpy=0 0 0 -> xyz=${rplidar_xoff} ${rplidar_yoff} ${rplidar_zoff} rpy=${pi} 0 ${-pi/2}

Commit message: fix: fix errors in lidar rotation link & jetson launch file

File: raspberryPI3/ros2_ws/src/geicar_description/src/description/geicar_description.urdf (robot description, URDF)
Before this commit: robot geicar, 18 links, 17 joints
Joints:
- joint rplidar_joint: origin xyz=${rplidar_xoff} ${rplidar_yoff} ${rplidar_zoff} rpy=${pi} 0 ${-pi/2} -> xyz=${rplidar_xoff} ${rplidar_yoff} ${rplidar_zoff} rpy=0 0 ${pi/2}

Commit message: fix: fix rotation of rplidar joint in robot description

File: raspberryPI3/ros2_ws/src/geicar_description/src/description/geicar_description.urdf (robot description, URDF)
Before this commit: robot geicar, 18 links, 17 joints
Joints:
- joint rplidar_joint: origin xyz=${rplidar_xoff} ${rplidar_yoff} ${rplidar_zoff} rpy=0 0 ${pi/2} -> xyz=${rplidar_xoff} ${rplidar_yoff} ${rplidar_zoff} rpy=0 0 ${rplidar_rotz}

Commit message: feat: Add node that converts cmd_vel(Twist) to a car command

File: raspberryPI3/ros2_ws/src/geicar_description/src/description/geicar_description.urdf (robot description, URDF)
Before this commit: robot geicar, 18 links, 17 joints
Links:
- link base_footprint: geometry visual box size=${base_length} ${base_width} ${base_height}
- link wheel_back_left_link: geometry visual cylinder length=${wheel_width} radius=${wheel_radius}
- link wheel_back_right_link: geometry visual cylinder length=${wheel_width} radius=${wheel_radius}
- link wheel_front_left_link: geometry visual cylinder length=${wheel_width} radius=${wheel_radius}
- link wheel_front_left_steer_link: geometry visual cylinder length=0.001 radius=0.01
- link wheel_front_right_link: geometry visual cylinder length=${wheel_width} radius=${wheel_radius}
Joints:
- joint wheel_back_right_joint: origin xyz=${-1*wheel_xoff} ${-1*wheel_yoff} ${wheel_zoff} rpy=0 0 0 -> xyz=-${wheel_xoff} -${wheel_yoff} ${wheel_zoff} rpy=0 0 0
