Commit message: fix: add joint limit to URDF & change name of default positions

File: jetsonNano/ros2_ws/src/ecosense_arm/config/ecosense_arm.ros2_control.xacro (robot description, xacro)
@@ -6,9 +6,9 @@
             <hardware>
                 <!-- By default, set up controllers for simulation. This won't work on real hardware -->
-                <!-- <plugin>mock_components/GenericSystem</plugin> -->
-                <plugin>so_arm_100_controller/SOARM100Interface</plugin>
-                <param name="use_serial">false</param>
+                <plugin>mock_components/GenericSystem</plugin>
+                <!-- <plugin>so_arm_100_controller/SOARM100Interface</plugin>
+                <param name="use_serial">true</param>
                 <param name="serial_port">/dev/ttyACM0</param>
-                <param name="serial_baudrate">1000000</param>
+                <param name="serial_baudrate">1000000</param> -->
             </hardware>
             <joint name="Shoulder_Rotation">

File: jetsonNano/ros2_ws/src/ecosense_arm/urdf/ecosense_arm.urdf (robot description, URDF)
Before this commit: robot ecosense_arm, 8 links, 7 joints
Links:
- removed link Base
- added link Arm_Base, mass 0.193184127927598; collision mesh filename=package://ecosense_arm/models/so_100_arm_5dof/meshes/Base.S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; visual mesh filename=package://ecosense_arm/models/so_100_arm_5dof/meshes/Base.S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
Joints:
- joint Elbow: limit (none) -> lower=-1.5708 upper=1.5708 effort=10.0 velocity=3.14; type continuous -> revolute
- joint Gripper: limit (none) -> lower=-0.17453292519 upper=1.5708 effort=10.0 velocity=3.14; type continuous -> revolute
- joint Shoulder_Pitch: limit (none) -> lower=-1.74532925199 upper=1.5708 effort=10.0 velocity=3.14; type continuous -> revolute
- joint Shoulder_Rotation: limit (none) -> lower=-1.5708 upper=1.5708 effort=10.0 velocity=3.14; origin xyz=0 -0.0452 0.0165 rpy=1.5708 0 0 -> xyz=0.0452 0 0.0165 rpy=1.5708 0 1.5708; parent Base -> Arm_Base; type continuous -> revolute
- joint Wrist_Pitch: limit (none) -> lower=-3.1416 upper=0 effort=10.0 velocity=3.14; type continuous -> revolute
- joint Wrist_Roll: limit (none) -> lower=-1.5708 upper=1.5708 effort=10.0 velocity=3.14; type continuous -> revolute
- joint base_link_joint: child Base -> Arm_Base

Commit message: feat: add arm to general URDF file and launch file

File: jetsonNano/ros2_ws/src/ecosense_arm/config/ecosense_arm.ros2_control.xacro (robot description, xacro)
@@ -1,5 +1,5 @@
 <?xml version="1.0"?>
 <robot xmlns:xacro="http://www.ros.org/wiki/xacro">
-    <xacro:macro name="ecosense_arm_ros2_control" params="name initial_positions_file">
+    <xacro:macro name="ecosense_arm_ros2_control" params="name initial_positions_file use_fake_hardware">
         <xacro:property name="initial_positions" value="${xacro.load_yaml(initial_positions_file)['initial_positions']}"/>
         <ros2_control name="${name}" type="system">

File: jetsonNano/ros2_ws/src/ecosense_arm/config/ecosense_arm.urdf.xacro (robot description, xacro)
@@ -2,8 +2,11 @@
 <robot xmlns:xacro="http://www.ros.org/wiki/xacro" name="ecosense_arm">
     <xacro:arg name="initial_positions_file" default="initial_positions.yaml" />
+    <xacro:arg name="use_fake_hardware" default="true" />
     <!-- Import ecosense_arm urdf file -->
-    <xacro:include filename="$(find ecosense_arm)/urdf/ecosense_arm.urdf" />
+    <xacro:include filename="$(find ecosense_arm)/urdf/ecosense_arm_world.urdf" />
     <!-- Import control_xacro -->
     <xacro:include filename="ecosense_arm.ros2_control.xacro" />
-    <xacro:ecosense_arm_ros2_control name="ECOSenseArm" initial_positions_file="$(arg initial_positions_file)"/>
+    <xacro:ecosense_arm_ros2_control name="ECOSenseArm"
+        initial_positions_file="$(arg initial_positions_file)"
+        use_fake_hardware="$(arg use_fake_hardware)"/>
 </robot>

File: jetsonNano/ros2_ws/src/ecosense_arm/urdf/ecosense_arm.urdf (robot description, URDF)
Before this commit: robot ecosense_arm, 8 links, 7 joints
Links:
- removed link Arm_Base
- removed link Fixed_Gripper
- removed link Lower_Arm
- removed link Moving_Jaw
- removed link Shoulder_Rotation_Pitch
- removed link Upper_Arm
- removed link Wrist_Pitch_Roll
- removed link base_link
Joints:
- removed joint Elbow
- removed joint Gripper
- removed joint Shoulder_Pitch
- removed joint Shoulder_Rotation
- removed joint Wrist_Pitch
- removed joint Wrist_Roll
- removed joint base_link_joint
