Commit message: fix: move robot description and robot state publisher to jetson to avoid bug when base_link is published after odom

File: jetsonNano/ros2_ws/src/ecosense_description/src/description/ecosense_description.urdf (robot description, URDF)
Before this commit: robot geicar, 18 links, 17 joints
Links:
- link base_footprint: geometry 
- link base_link: geometry visual box size=${base_length} ${base_width} ${base_height}

Commit message: fix: fix cameras frame to fit with ROS Standard

File: jetsonNano/ros2_ws/src/ecosense_description/src/description/ecosense_description.urdf (robot description, URDF)
Before this commit: robot ecosense, 18 links, 17 joints
Joints:
- joint camera_left_joint: origin xyz=${camera_left_xoff} ${camera_left_yoff} ${camera_left_zoff} rpy=0 0 0 -> xyz=${camera_left_xoff} ${camera_left_yoff} ${camera_left_zoff} rpy=${camera_left_rotx} ${camera_left_roty} ${camera_left_rotz}
- joint camera_right_joint: origin xyz=${camera_right_xoff} ${camera_right_yoff} ${camera_right_zoff} rpy=0 0 0 -> xyz=${camera_right_xoff} ${camera_right_yoff} ${camera_right_zoff} rpy=${camera_right_rotx} ${camera_right_roty} ${camera_right_rotz}; parent base_link -> camera_left_link

Commit message: feat: add new LD lidar to URDF

File: jetsonNano/ros2_ws/src/ecosense_description/src/description/ecosense_description.urdf (robot description, URDF)
Before this commit: robot ecosense, 18 links, 17 joints
Links:
- added link ld_lidar_link
Joints:
- added joint ld_lidar_joint: type fixed, parent base_link, child ld_lidar_link, origin xyz=${ld_lidar_xoff} ${ld_lidar_yoff} ${ld_lidar_zoff} rpy=0 0 0

Commit message: fix: change description to add constant

File: jetsonNano/ros2_ws/src/ecosense_description/src/description/ecosense_description.urdf (robot description, URDF)
Before this commit: robot ecosense, 19 links, 18 joints
Joints:
- joint ld_lidar_joint: origin xyz=${ld_lidar_xoff} ${ld_lidar_yoff} ${ld_lidar_zoff} rpy=0 0 0 -> xyz=${ld_lidar_xoff} ${ld_lidar_yoff} ${ld_lidar_zoff} rpy=${ld_lidar_rotx} ${ld_lidar_roty} ${ld_lidar_rotz}
