File: Pwr/hardware/pcb/cpu.kicad_sch (KiCad schematic)
At the start: 5 parts, among them J10 Conn_ARM_JTAG_SWD_10, SW1 SW_Push, U1 STM32C071F8Px

Commit message: WIP boitire PWR fini
Parts:
- added J2: FFC2B35-10-T, FFC2B3510T, symbol FFC2B35-10-T:FFC2B35-10-T
- added J3: 114020164, Grove 114020164:SEEEDSTUDIO_114020164, symbol Grove 114020164:114020164
- added LS1: PS1240P02CT3, Buzzer_TDK:PS1240P02BT, symbol PS1240P02CT3:PS1240P02CT3
- added Q6: PMF250XNEX, Package_TO_SOT_SMD:SOT-323_SC-70, symbol Device:Q_NMOS_GSD
- added R14: 470R, Resistor_SMD:R_0805_2012Metric, symbol Device:R
- added R15: 10K, Resistor_SMD:R_0805_2012Metric, symbol Device:R
- added R2, R3: 4.7K, Resistor_SMD:R_0805_2012Metric, symbol Device:R
Connections:
- net GND: now also J2.3, J2.5, J3.4, Q6.2 (S), R15.2
- net OBC_SHUTDOWN: now also J3.3
- net RED_LED: now also J2.7
- net DISPLAY_CMD_DATA: no longer names the net of U1.2 (PC14)
- net DISPLAY_RESET: no longer names the net of U1.3 (PC15)
- net GREEN_LED renamed BUZZER
- net BUZZER: now also R14.1
- net I2C_SCL renamed I2C1_SCL
- net I2C1_SCL: now also J3.1, R3.2
- net I2C_SDA renamed I2C1_SDA
- net I2C1_SDA: now also J3.2, R2.2
- net SPI_MOSI renamed SPI1_MOSI
- net SPI1_MOSI: now also J2.4
- net SPI_NSS renamed SPI1_NSS
- net SPI1_NSS: now also J2.6
- net SPI_SCK renamed SPI1_SCK
- net SPI1_SCK: now also J2.2
- new net: Q6.1 (G), R14.2, R15.1
- new net: LS1.1, Q6.3 (D)
- new net +3.3V: LS1.2
- new net +3.3V_Ecran: J2.1, R2.1, R3.1
- no-connect marks 2 -> 9
Other:
- note added: "<- Attention: on parle bien du 3v3/6A produit par le module DC/DC buck, pas du 3v3 MCU ou 3v3 ecran, faible amperage generé par le petit regulateur LDO"
- note added: "Ne pas installer"
- moved on the sheet: C1, R8, SW1, U1
