File: Pwr/hardware/pcb/pwr.kicad_pcb (KiCad board)
At the start: 4 copper layers, 100 x 70 mm, 51 parts, among them J1 XT60PW-M, J10 Conn_ARM_JTAG_SWD_10, J11 Conn_01x06, J12 Conn_01x06, J13 Conn_01x06, J14 Conn_01x06, J2 FFC2B35-10-T, J3 114020164, J4 XT60, J5 Conn_01x02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

Commit message: WIP boitire PWR fini
Parts:
- added LS1: PS1240P02CT3, Buzzer_TDK:PS1240P02BT, F.Cu at (108.0, 91.8)
- added Q6: PMF250XNEX, Package_TO_SOT_SMD:SOT-323_SC-70, F.Cu at (188.0, 70.5)
- added R14: 470R, Resistor_SMD:R_0805_2012Metric, F.Cu at (184.0, 70.4)
- added R15: 10K, Resistor_SMD:R_0805_2012Metric, F.Cu at (188.0, 76.0)
- J6, J7: moved to B.Cu
- moved J7 21.7 mm to (195.5, 69.8)
- moved J6 21.6 mm to (104.8, 69.8)
- moved R7 18.6 mm to (150.8, 55.0), turned to 180 degrees
- moved F1 11.0 mm to (140.0, 66.5), turned to 90 degrees
- moved J2 9.51 mm to (168.0, 81.0), turned to 180 degrees
- moved Q3 7.91 mm to (167.0, 71.3)
- moved R4 7.91 mm to (170.4, 71.3)
- moved Q1 6.74 mm to (151.0, 63.9), turned to -90 degrees
- moved R2 4.60 mm to (190.0, 86.4), turned to -90 degrees
- moved C1 3.59 mm to (184.0, 66.0)
- moved PS5 3.47 mm to (127.5, 109.0)
- moved SW1 3.29 mm to (106.0, 105.2), turned to 180 degrees
- moved R8 2.98 mm to (108.2, 101.0), turned to 0 degrees
- moved Q2 2.75 mm to (148.0, 75.8)
- moved R1 2.75 mm to (152.5, 74.2)
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Connections:
- J2 pad 1: +3.3V -> +3.3V_Ecran
- J2 pad 10: /Ecran - I2C - Divers/GREEN_LED -> unconnected-(J2-Pad10)
- J2 pad 6: /CPU - Debug/DISPLAY_RESET -> /CPU - Debug/SPI1_NSS
- J2 pad 7: /CPU - Debug/DISPLAY_CMD_DATA -> /CPU - Debug/RED_LED
- J2 pad 8: /CPU - Debug/SPI1_NSS -> unconnected-(J2-Pad8)
- J2 pad 9: /Ecran - I2C - Divers/RED_LED -> unconnected-(J2-Pad9)
- R2 pad 2: /CPU - Debug/I2C1_SCL -> /CPU - Debug/I2C1_SDA
- R3 pad 2: /CPU - Debug/I2C1_SDA -> /CPU - Debug/I2C1_SCL
- U1 pad 17: /CPU - Debug/GREEN_LED -> /CPU - Debug/BUZZER
- U1 pad 2: /CPU - Debug/DISPLAY_CMD_DATA -> unconnected-(U1-PC14-Pad2)
- U1 pad 3: /CPU - Debug/DISPLAY_RESET -> unconnected-(U1-PC15-Pad3)
Other:
- outline, holes or cut-outs redrawn
