File: Pwr/hardware/pcb/pwr.kicad_sch (KiCad schematic)
At the start: 4 parts

Commit message: WIP boitire PWR fini
Other:
- removed sheet Ecran - I2C - Divers
- sheet CPU - Debug ports: added none; removed DISPLAY_CMD_DATA, DISPLAY_RESET, GREEN_LED, I2C_SCL, I2C_SDA, OBC_SHUTDOWN, RED_LED, SPI_MOSI, SPI_NSS, SPI_SCK
