File: Pwr/hardware/pcb/pcb-ecran/pcb-ecran.kicad_sch (KiCad schematic)
At the start: 8 parts, among them J2 FFC2B35-10-T, U3 DM-OLED096-636

Commit message: WIP boitire PWR fini
Parts:
- removed D2: APT2012LSECK/J3-PRV, LED_SMD:LED_0805_2012Metric, symbol Device:LED
- removed H5, H6, H7, H8: MountingHole, MountingHole:MountingHole_3.2mm_M3, symbol Mechanical:MountingHole
- removed J2: FFC2B35-10-T, FFC2B3510T, symbol FFC2B35-10-T:FFC2B35-10-T
- removed R5: 1K, Resistor_SMD:R_0805_2012Metric, symbol Device:R
- removed U3: DM-OLED096-636, oled-0.96:MODULE_DM-OLED096-636, symbol DM-OLED096-636:DM-OLED096-636
- added D1: APT2012LSECK/J3-PRV, LED_SMD:LED_0805_2012Metric, symbol Device:LED
- added H1, H2, H3, H4: MountingHole, MountingHole:MountingHole_3.2mm_M3, symbol Mechanical:MountingHole
- added J1: FFC2B35-10-T, FFC2B3510T, symbol FFC2B35-10-T:FFC2B35-10-T
- added R1: 1K, Resistor_SMD:R_0805_2012Metric, symbol Device:R
- added U1: DM-OLED096-636, oled-0.96:MODULE_DM-OLED096-636, symbol DM-OLED096-636:DM-OLED096-636
Connections:
- net +3.3V_Ecran: now also J1.1, U1.2 (VCC_IN)
- net GND: now also J1.3, J1.5, R1.2, U1.1 (GND)
- net RED_LED: now also D1.2 (A), J1.7
- net SPI_DATA: now also J1.4, U1.4 (SDA)
- net SPI_SCK: now also J1.2, U1.3 (SCL)
- net ~{SPI_CS}: now also J1.6
- new net: D1.1 (K), R1.1
Other:
- company: INSA - GEI -> (none)
- title: Carte Energie - I/O -> (none)
