File: Pwr/hardware/pcb v2/cpu.kicad_sch (KiCad schematic)
At the start: 16 parts, among them J10 Conn_ARM_JTAG_SWD_10, J2 FFC2B35-10-T, J3 114020164, Q6 PMF250XNEX, U1 STM32C071F8Px

Commit message: Correction sur l'ecran SPI
Connections:
- net DISPLAY_CD: now reaches U1.2 (PC14)
- net DISPLAY_CD: now also J2.8
- net DISPLAY_RESET: now reaches U1.3 (PC15)
- net DISPLAY_RESET: now also J2.7
- no-connect marks 10 -> 6
Changed lines of the file:
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@@
-	)
-	(no_connect
-		(at 129.54 167.64)
 	)
 	(no_connect
@@
 	)
 	(no_connect
-		(at 109.22 82.55)
-	)
-	(no_connect
 		(at 154.94 152.4)
-	)
-	(no_connect
-		(at 129.54 170.18)
 	)
 	(no_connect
@@
 		(at 154.94 154.94)
 	)
-	(no_connect
-		(at 109.22 80.01)
-	)
 	(wire
 		(pts
@@
 	(wire
 		(pts
+			(xy 107.95 167.64) (xy 129.54 167.64)
+		)
+		(stroke
+			(width 0)
+			(type default)
+		)
+	)
+	(wire
+		(pts
+			(xy 88.9 82.55) (xy 109.22 82.55)
+		)
+		(stroke
+			(width 0)
+			(type default)
+		)
+	)
+	(wire
+		(pts
 			(xy 71.12 111.76) (xy 71.12 116.84)
 		)
@@
 	(wire
 		(pts
+			(xy 88.9 80.01) (xy 109.22 80.01)
+		)
+		(stroke
+			(width 0)
+			(type default)
+		)
+	)
+	(wire
+		(pts
 			(xy 160.02 90.17) (xy 184.15 90.17)
 		)
@@
 		(pts
 			(xy 252.73 132.08) (xy 242.57 132.08)
+		)
+		(stroke
+			(width 0)
+			(type default)
+		)
+	)
+	(wire
+		(pts
+			(xy 107.95 170.18) (xy 129.54 170.18)
 		)
 		(stroke
@@
 		)
 	)
+	(label "DISPLAY_RESET"
+		(at 88.9 82.55 0)
+		(effects
+			(font
+				(size 1.27 1.27)
+			)
+			(justify left bottom)
+		)
+	)
 	(label "SCREEN_PMOS_ENABLE"
 		(at 184.15 95.25 180)
@@
 		)
 	)
+	(label "DISPLAY_CD"
+		(at 107.95 170.18 0)
+		(effects
+			(font
+				(size 1.27 1.27)
+			)
+			(justify left bottom)
+		)
+	)
 	(label "DEBUG_SWCLK"
 		(at 180.34 105.41 180)
@@
 		)
 	)
+	(label "DISPLAY_CD"
+		(at 88.9 80.01 0)
+		(effects
+			(font
+				(size 1.27 1.27)
+			)
+			(justify left bottom)
+		)
+	)
 	(label "~{nRESET}"
 		(at 88.9 74.93 0)
@@
 		)
 	)
+	(label "DISPLAY_RESET"
+		(at 107.95 167.64 0)
+		(effects
+			(font
+				(size 1.27 1.27)
+			)
+			(justify left bottom)
+		)
+	)
