File: IO/hardware/carte-io (prochaine version)/int_sensors.kicad_sch (KiCad schematic)
At the start: 12 parts, among them U12 LSM6DS3, U13 LIS2MDL, U14 LPS22DF, U18 APDS-9251-001, U19 SHT4x

Commit message: Recuperation de la carte IO perdue lors de la suppression des 3 derniers commit
Other:
- note added: "A installer. Ce bus I2C vient du MCU et aucune resitance n'est presente"
Changed lines of the file:
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@@
+		)
+	)
+	(rectangle
+		(start 43.18 27.94)
+		(end 68.58 38.1)
+		(stroke
+			(width 0)
+			(type default)
+		)
+		(fill
+			(type none)
+		)
+	)
+	(text "A installer. Ce bus I2C vient du MCU\net aucune resitance n'est presente"
+		(exclude_from_sim no)
+		(at 69.596 33.274 0)
+		(effects
+			(font
+				(size 1.27 1.27)
+			)
+			(justify left)
 		)
 	)
@@
 			)
 		)
-		(property "Description" "Digital Humidity and Temperature Sensor, +/-1%RH, +/-0.1degC, I2C, 1.08-3.6V, 16bit, DFN-4"
+		(property "Description" "Digital Humidity and Temperature Sensor, ±1%RH, ±0.1°C, I2C, 1.08-3.6V, 16bit, DFN-4"
 			(at 67.31 80.01 0)
 			(effects
